File: carte elec/carte elec.kicad_pcb (KiCad board)
At the start: 2 copper layers, 75 x 88.5 mm, 55 parts, among them J1 SD_Card_Device, J2 Barrel_Jack_Switch, U1 ESP32-S3-UNO, U2 R-78E5.0-1.0

Commit message: fix wiring problems
Parts:
- moved D1 63.7 mm to (42.0, 127.5)
- moved R11 59.8 mm to (42.0, 122.5), turned to -90 degrees
- moved C11 3.54 mm to (98.5, 110.0)
Connections:
- C11 pad 1: +5V -> +12V
- U1 pad 8: +5V -> +12V
Routing:
- net +5V: track 139.9 -> 45.5 mm
- net +12V: track 74.0 -> 140.4 mm
- net Net-(D1-A): track 3.18 -> 2.60 mm
