File: carte elec/carte elec.kicad_sch (KiCad schematic)
At the start: 55 parts, among them J1 SD_Card_Device, J2 Barrel_Jack_Switch, U1 ESP32-S3-UNO, U2 R-78E5.0-1.0

Commit message: fix wiring problems
Parts:
- renumbered down to down1, left to left1, right to right1
Connections:
- net +12V: now also C11.1, U1.8 (VIN)
- net +5V: no longer C11.1, U1.8 (VIN)
